Commit message: Step:3 gripper draft

File: src/Universal_Robots_ROS2_Description/urdf/ur_macro.xacro (robot description, xacro)
@@ -433,5 +433,5 @@
       <parent link="${tf_prefix}flange"/>
       <child link="${tf_prefix}gripper"/>
-      <origin xyz="0 0 0.1" rpy="0 0 0"/>
+      <origin xyz="0.1 0 0" rpy="0 ${pi/2} 0"/>
     </joint>
   </xacro:macro>
